File: circuit_board/ltm-ps.sch (KiCad schematic (older format))
At the start: 19 parts, among them P1 CONN_01X02, P2 CONN_01X02, P3 CONN_01X02, U1 NCP1092, U2 LTM8050

Commit message: add ncp1092 resistors settings comments
Other:
- note added: "- R3 sets the detection current regulation\nduring PoE detection phase. It is set by the\nmanufacturer (see NCP1092 datasheet)\n- R4 sets the PoE class. Datashett gives\nresistance values for each class. 4.42k is for\nclass 0 (13W)\n- R5 sets the inrush current limit"
- moved on the sheet: U2B
Changed lines of the file:
@@
-EESchema Schematic File Version 2  date Mon 02 Feb 2015 02:27:46 PM CET
+EESchema Schematic File Version 2  date Mon 02 Feb 2015 03:01:30 PM CET
 LIBS:power
 LIBS:device
@@
 Comment4 ""
 $EndDescr
+Text Notes 4500 4100 0    60   ~ 12
+- R3 sets the detection current regulation\nduring PoE detection phase. It is set by the\nmanufacturer (see NCP1092 datasheet)\n- R4 sets the PoE class. Datashett gives\nresistance values for each class. 4.42k is for\nclass 0 (13W)\n- R5 sets the inrush current limit
 Text Label 1750 950  2    60   ~ 0
 VAUX
@@
 Wire Wire Line
 	7350 3350 6450 3350
-Connection ~ 4800 6350
-Wire Wire Line
-	4800 6400 4800 5250
-Wire Wire Line
-	5850 6850 5850 7100
+Connection ~ 5300 6900
+Wire Wire Line
+	5300 6950 5300 5800
+Wire Wire Line
+	6350 7400 6350 7650
 Wire Wire Line
 	8100 3450 7450 3450
@@
 Wire Wire Line
 	2350 4050 2200 4050
-Connection ~ 5750 4550
-Wire Wire Line
-	5750 4550 5750 4750
-Connection ~ 5950 4550
-Wire Wire Line
-	5950 4550 5950 4750
-Wire Wire Line
-	6150 4750 6150 4550
-Wire Wire Line
-	5550 4750 5550 4550
-Connection ~ 4800 5550
-Wire Wire Line
-	4800 5550 5000 5550
-Connection ~ 4800 5350
-Wire Wire Line
-	4800 5350 5000 5350
-Connection ~ 4800 5850
-Wire Wire Line
-	4800 5850 5000 5850
-Connection ~ 4800 6050
-Wire Wire Line
-	4800 6050 5000 6050
-Connection ~ 4800 6250
-Wire Wire Line
-	4800 6250 5000 6250
-Connection ~ 6900 5400
-Wire Wire Line
-	6900 5400 6700 5400
-Connection ~ 6900 5600
-Wire Wire Line
-	6900 5600 6700 5600
-Connection ~ 6900 5800
-Wire Wire Line
-	6900 5800 6700 5800
-Connection ~ 6900 6000
-Wire Wire Line
-	6900 6000 6700 6000
-Connection ~ 6900 6200
-Wire Wire Line
-	6900 6200 6700 6200
-Connection ~ 5650 7050
-Wire Wire Line
-	5650 6850 5650 7050
-Connection ~ 6050 7050
-Wire Wire Line
-	6050 6850 6050 7050
-Wire Wire Line
-	5550 6850 5550 7050
+Connection ~ 6250 5100
+Wire Wire Line
+	6250 5100 6250 5300
+Connection ~ 6450 5100
+Wire Wire Line
+	6450 5100 6450 5300
+Wire Wire Line
+	6650 5300 6650 5100
+Wire Wire Line
+	6050 5300 6050 5100
+Connection ~ 5300 6100
+Wire Wire Line
+	5300 6100 5500 6100
+Connection ~ 5300 5900
+Wire Wire Line
+	5300 5900 5500 5900
+Connection ~ 5300 6400
+Wire Wire Line
+	5300 6400 5500 6400
+Connection ~ 5300 6600
+Wire Wire Line
+	5300 6600 5500 6600
+Connection ~ 5300 6800
+Wire Wire Line
+	5300 6800 5500 6800
+Connection ~ 7400 5950
+Wire Wire Line
+	7400 5950 7200 5950
+Connection ~ 7400 6150
+Wire Wire Line
+	7400 6150 7200 6150
+Connection ~ 7400 6350
+Wire Wire Line
+	7400 6350 7200 6350
+Connection ~ 7400 6550
+Wire Wire Line
+	7400 6550 7200 6550
+Connection ~ 7400 6750
+Wire Wire Line
+	7400 6750 7200 6750
+Connection ~ 6150 7600
+Wire Wire Line
+	6150 7400 6150 7600
+Connection ~ 6550 7600
+Wire Wire Line
+	6550 7400 6550 7600
+Wire Wire Line
+	6050 7400 6050 7600
 Wire Wire Line
 	8100 3050 7950 3050
@@
 	7450 2950 8100 2950
 Wire Wire Line
-	5550 7050 6150 7050
-Wire Wire Line
-	6150 7050 6150 6850
-Connection ~ 5850 7050
-Wire Wire Line
-	5950 7050 5950 6850
-Connection ~ 5950 7050
-Wire Wire Line
-	5750 7050 5750 6850
-Connection ~ 5750 7050
-Wire Wire Line
-	6700 5300 6900 5300
-Wire Wire Line
-	6900 6300 6700 6300
-Wire Wire Line
-	6900 6100 6700 6100
-Connection ~ 6900 6100
-Wire Wire Line
-	6900 5900 6700 5900
-Connection ~ 6900 5900
-Wire Wire Line
-	6900 5700 6700 5700
-Connection ~ 6900 5700
-Wire Wire Line
-	6900 5500 6700 5500
-Connection ~ 6900 5500
-Wire Wire Line
-	4800 5250 5000 5250
-Wire Wire Line
-	4800 6350 5000 6350
-Wire Wire Line
-	4800 6150 5000 6150
-Connection ~ 4800 6150
-Wire Wire Line
-	4800 5950 5000 5950
-Connection ~ 4800 5950
-Wire Wire Line
-	4800 5750 5000 5750
-Connection ~ 4800 5750
-Wire Wire Line
-	4800 5450 5000 5450
-Connection ~ 4800 5450
-Wire Wire Line
-	4800 5650 5000 5650
-Connection ~ 4800 5650
-Wire Wire Line
-	6050 4550 6050 4750
-Connection ~ 6050 4550
-Connection ~ 5850 4550
-Wire Wire Line
-	5650 4550 5650 4750
-Connection ~ 5650 4550
+	6050 7600 6650 7600
+Wire Wire Line
+	6650 7600 6650 7400
+Connection ~ 6350 7600
+Wire Wire Line
+	6450 7600 6450 7400
+Connection ~ 6450 7600
+Wire Wire Line
+	6250 7600 6250 7400
+Connection ~ 6250 7600
+Wire Wire Line
+	7200 5850 7400 5850
+Wire Wire Line
+	7400 6850 7200 6850
+Wire Wire Line
+	7400 6650 7200 6650
+Connection ~ 7400 6650
+Wire Wire Line
+	7400 6450 7200 6450
+Connection ~ 7400 6450
+Wire Wire Line
+	7400 6250 7200 6250
+Connection ~ 7400 6250
+Wire Wire Line
+	7400 6050 7200 6050
+Connection ~ 7400 6050
+Wire Wire Line
+	5300 5800 5500 5800
+Wire Wire Line
+	5300 6900 5500 6900
+Wire Wire Line
+	5300 6700 5500 6700
+Connection ~ 5300 6700
+Wire Wire Line
+	5300 6500 5500 6500
+Connection ~ 5300 6500
+Wire Wire Line
+	5300 6300 5500 6300
+Connection ~ 5300 6300
+Wire Wire Line
+	5300 6000 5500 6000
+Connection ~ 5300 6000
+Wire Wire Line
+	5300 6200 5500 6200
+Connection ~ 5300 6200
+Wire Wire Line
+	6550 5100 6550 5300
+Connection ~ 6550 5100
+Connection ~ 6350 5100
+Wire Wire Line
+	6150 5100 6150 5300
+Connection ~ 6150 5100
 Wire Wire Line
 	6550 3450 6550 3550
@@
 Connection ~ 3900 950
 Wire Wire Line
-	5550 4550 6150 4550
-Wire Wire Line
-	6900 5300 6900 6350
-Connection ~ 6900 6300
-Wire Wire Line
-	5850 4500 5850 4750
+	6050 5100 6650 5100
+Wire Wire Line
+	7400 5850 7400 6900
+Connection ~ 7400 6850
+Wire Wire Line
+	6350 5050 6350 5300
 Wire Wire Line
 	3700 2550 3700 2500
@@
 L GND #PWR03
 U 1 1 54CF696E
-P 5850 4500
-F 0 "#PWR03" H 5850 4250 60  0001 C CNN
-F 1 "GND" H 5850 4350 60  0000 C CNN
-	1    5850 4500
+P 6350 5050
+F 0 "#PWR03" H 6350 4800 60  0001 C CNN
+F 1 "GND" H 6350 4900 60  0000 C CNN
+	1    6350 5050
 	-1   0    0    1
 $EndComp
@@
 L GND #PWR04
 U 1 1 54CF6965
-P 4800 6400
-F 0 "#PWR04" H 4800 6150 60  0001 C CNN
-F 1 "GND" H 4800 6250 60  0000 C CNN
-	1    4800 6400
+P 5300 6950
+F 0 "#PWR04" H 5300 6700 60  0001 C CNN
+F 1 "GND" H 5300 6800 60  0000 C CNN
+	1    5300 6950
 	1    0    0    -1
 $EndComp
@@
 L GND #PWR05
 U 1 1 54CF6961
-P 6900 6350
-F 0 "#PWR05" H 6900 6100 60  0001 C CNN
-F 1 "GND" H 6900 6200 60  0000 C CNN
-	1    6900 6350
+P 7400 6900
+F 0 "#PWR05" H 7400 6650 60  0001 C CNN
+F 1 "GND" H 7400 6750 60  0000 C CNN
+	1    7400 6900
 	1    0    0    -1
 $EndComp
@@
 L GND #PWR013
 U 1 1 54CCC93A
-P 5850 7100
-F 0 "#PWR013" H 5850 6850 60  0001 C CNN
-F 1 "GND" H 5850 6950 60  0000 C CNN
-	1    5850 7100
+P 6350 7650
+F 0 "#PWR013" H 6350 7400 60  0001 C CNN
+F 1 "GND" H 6350 7500 60  0000 C CNN
+	1    6350 7650
 	1    0    0    -1
 $EndComp
@@
 L LTM8050 U2
 U 2 1 54C96618
-P 5850 5800
-F 0 "U2" H 5350 6600 60  0000 C CNN
-F 1 "LTM8050" H 5850 5800 60  0000 C CNN
-	2    5850 5800
-	1    0    0    -1
-$EndComp
+P 6350 6350
+F 0 "U2" H 5850 7150 60  0000 C CNN
+F 1 "LTM8050" H 6350 6350 60  0000 C CNN
+	2    6350 6350
+	1    0    0    -1
+$EndComp

Commit message: add RJ45 PoE component in schematic
Parts:
- added J1: GIGABIT_MAGJACK, symbol GIGABIT_MAGJACK
Connections:
- no-connect marks 2 -> 6
Changed lines of the file:
@@
-EESchema Schematic File Version 2  date Mon 02 Feb 2015 03:01:30 PM CET
+EESchema Schematic File Version 2  date Tue 03 Feb 2015 05:19:26 PM CET
 LIBS:power
 LIBS:device
@@
 Sheet 1 1
 Title ""
-Date "2 feb 2015"
+Date "3 feb 2015"
 Rev ""
 Comp ""
@@
 Comment4 ""
 $EndDescr
+NoConn ~ 1000 7250
+NoConn ~ 1000 7150
+NoConn ~ 3350 7250
+NoConn ~ 3350 7150
+$Comp
+L GIGABIT_MAGJACK J1
+U 1 1 54D0F1C7
+P 2200 6100
+F 0 "J1" H 1400 7400 60  0000 C CNN
+F 1 "GIGABIT_MAGJACK" H 2250 4800 60  0000 C CNN
+	1    2200 6100
+	-1   0    0    1
+$EndComp
 Text Notes 4500 4100 0    60   ~ 12
 - R3 sets the detection current regulation\nduring PoE detection phase. It is set by the\nmanufacturer (see NCP1092 datasheet)\n- R4 sets the PoE class. Datashett gives\nresistance values for each class. 4.42k is for\nclass 0 (13W)\n- R5 sets the inrush current limit
@@
 vout_5V@2A
 $Comp
-L PWR_FLAG #FLG01
+L PWR_FLAG #FLG3
 U 1 1 54CF6F79
 P 2000 3400
-F 0 "#FLG01" H 2000 3495 30  0001 C CNN
+F 0 "#FLG3" H 2000 3495 30  0001 C CNN
 F 1 "PWR_FLAG" H 2000 3580 30  0000 C CNN
 	1    2000 3400
@@
 $EndComp
 $Comp
-L PWR_FLAG #FLG02
+L PWR_FLAG #FLG4
 U 1 1 54CF6F68
 P 3700 2500
-F 0 "#FLG02" H 3700 2595 30  0001 C CNN
+F 0 "#FLG4" H 3700 2595 30  0001 C CNN
 F 1 "PWR_FLAG" H 3700 2680 30  0000 C CNN
 	1    3700 2500
@@
 For the prototype version, this jumper allows to select\nwhich signal will enable the DC/DC converter.\n- NCP1092 PGOOD\n- VIN (VPORT_P/Auxiliary source)
 $Comp
-L GND #PWR03
+L GND #PWR6
 U 1 1 54CF696E
 P 6350 5050
-F 0 "#PWR03" H 6350 4800 60  0001 C CNN
+F 0 "#PWR6" H 6350 4800 60  0001 C CNN
 F 1 "GND" H 6350 4900 60  0000 C CNN
 	1    6350 5050
@@
 $EndComp
 $Comp
-L GND #PWR04
+L GND #PWR5
 U 1 1 54CF6965
 P 5300 6950
-F 0 "#PWR04" H 5300 6700 60  0001 C CNN
+F 0 "#PWR5" H 5300 6700 60  0001 C CNN
 F 1 "GND" H 5300 6800 60  0000 C CNN
 	1    5300 6950
@@
 $EndComp
 $Comp
-L GND #PWR05
+L GND #PWR9
 U 1 1 54CF6961
 P 7400 6900
-F 0 "#PWR05" H 7400 6650 60  0001 C CNN
+F 0 "#PWR9" H 7400 6650 60  0001 C CNN
 F 1 "GND" H 7400 6750 60  0000 C CNN
 	1    7400 6900
@@
 $EndComp
 $Comp
-L GND #PWR06
+L GND #PWR10
 U 1 1 54CF363A
 P 7450 3600
-F 0 "#PWR06" H 7450 3350 60  0001 C CNN
+F 0 "#PWR10" H 7450 3350 60  0001 C CNN
 F 1 "GND" H 7450 3450 60  0000 C CNN
 	1    7450 3600
@@
 VAUX
 $Comp
-L GND #PWR07
+L GND #PWR14
 U 1 1 54CF3305
 P 10550 5500
-F 0 "#PWR07" H 10550 5250 60  0001 C CNN
+F 0 "#PWR14" H 10550 5250 60  0001 C CNN
 F 1 "GND" H 10550 5350 60  0000 C CNN
 	1    10550 5500
@@
 $EndComp
 $Comp
-L GND #PWR08
+L GND #PWR13
 U 1 1 54CF32E7
 P 10550 4800
-F 0 "#PWR08" H 10550 4550 60  0001 C CNN
+F 0 "#PWR13" H 10550 4550 60  0001 C CNN
 F 1 "GND" H 10550 4650 60  0000 C CNN
 	1    10550 4800
@@
 $EndComp
 $Comp
-L GND #PWR09
+L GND #PWR12
 U 1 1 54CF3238
 P 8750 1550
-F 0 "#PWR09" H 8750 1300 60  0001 C CNN
+F 0 "#PWR12" H 8750 1300 60  0001 C CNN
 F 1 "GND" H 8750 1400 60  0000 C CNN
 	1    8750 1550
@@
 $EndComp
 $Comp
-L GND #PWR010
+L GND #PWR4
 U 1 1 54CF3233
 P 4950 1550
-F 0 "#PWR010" H 4950 1300 60  0001 C CNN
+F 0 "#PWR4" H 4950 1300 60  0001 C CNN
 F 1 "GND" H 4950 1400 60  0000 C CNN
 	1    4950 1550
@@
 AUX
 $Comp
-L GND #PWR011
+L GND #PWR3
 U 1 1 54CF3016
 P 1950 2250
-F 0 "#PWR011" H 1950 2000 60  0001 C CNN
+F 0 "#PWR3" H 1950 2000 60  0001 C CNN
 F 1 "GND" H 1950 2100 60  0000 C CNN
 	1    1950 2250
@@
 $EndComp
 $Comp
-L GND #PWR012
+L GND #PWR8
 U 1 1 54CCE0E0
 P 6550 3550
-F 0 "#PWR012" H 6550 3300 60  0001 C CNN
+F 0 "#PWR8" H 6550 3300 60  0001 C CNN
 F 1 "GND" H 6550 3400 60  0000 C CNN
 	1    6550 3550
@@
 $EndComp
 $Comp
-L GND #PWR013
+L GND #PWR7
 U 1 1 54CCC93A
 P 6350 7650
-F 0 "#PWR013" H 6350 7400 60  0001 C CNN
+F 0 "#PWR7" H 6350 7400 60  0001 C CNN
 F 1 "GND" H 6350 7500 60  0000 C CNN
 	1    6350 7650
@@
 NoConn ~ 8100 3250
 $Comp
-L GND #PWR014
+L GND #PWR11
 U 1 1 54CCC8D2
 P 7800 4350
-F 0 "#PWR014" H 7800 4100 60  0001 C CNN
+F 0 "#PWR11" H 7800 4100 60  0001 C CNN
 F 1 "GND" H 7800 4200 60  0000 C CNN
 	1    7800 4350
@@
 $EndComp
 $Comp
-L GND #PWR015
+L GND #PWR2
 U 1 1 54C01912
 P 1350 1550
-F 0 "#PWR015" H 1350 1300 60  0001 C CNN
+F 0 "#PWR2" H 1350 1300 60  0001 C CNN
 F 1 "GND" H 1350 1400 60  0000 C CNN
 	1    1350 1550
@@
 $EndComp
 $Comp
-L PWR_FLAG #FLG016
+L PWR_FLAG #FLG2
 U 1 1 54C0190D
 P 1350 1500
-F 0 "#FLG016" H 1350 1595 30  0001 C CNN
+F 0 "#FLG2" H 1350 1595 30  0001 C CNN
 F 1 "PWR_FLAG" H 1350 1680 30  0000 C CNN
 	1    1350 1500
@@
 $EndComp
 $Comp
-L PWR_FLAG #FLG017
+L PWR_FLAG #FLG1
 U 1 1 54C01907
 P 1350 850
-F 0 "#FLG017" H 1350 945 30  0001 C CNN
+F 0 "#FLG1" H 1350 945 30  0001 C CNN
 F 1 "PWR_FLAG" H 1350 1030 30  0000 C CNN
 	1    1350 850
@@
 $EndComp
 $Comp
-L GND #PWR018
+L GND #PWR1
 U 1 1 54C018EC
 P 1050 1050
-F 0 "#PWR018" H 1050 800 60  0001 C CNN
+F 0 "#PWR1" H 1050 800 60  0001 C CNN
 F 1 "GND" H 1050 900 60  0000 C CNN
 	1    1050 1050
