File: circuit_board/ltm-ps.sch (KiCad schematic (older format))
At the start: 20 parts, among them J1 GIGABIT_MAGJACK, P1 CONN_01X02, P2 CONN_01X02, P3 CONN_01X02, U1 NCP1092, U2 LTM8050

Commit message: add RJ45 out connector and some comments
Parts:
- added C3: 1000p, symbol C
- added J2: RJHSE-5080, symbol RJ45
- added R10, R11, R8, R9: 75R, symbol R
- D4: value TVS -> SMAJ58CA
- J1: value GIGABIT_MAGJACK -> 0826-1X1T-M1-F
Connections:
- net labels added: TRD1+, TRD1-, TRD2+, TRD2-, TRD3+, TRD3-, TRD4+, TRD4-, VPoE_1+, VPoE_1-, VPoE_2+, VPoE_2-
- wire segments 134 -> 177
- no-connect marks 6 -> 7
Other:
- note added: "1kV"
- note added: "DigiKey - 380-1122-ND"
- note added: "Farnell - 1860577"
- moved on the sheet: D1, P1, U1, U2A, U2B, U2C, U2D
