File: circuit_board/ltm-ps.sch (KiCad schematic (older format))
At the start: 26 parts, among them J1 0826-1X1T-M1-F, J2 RJHSE-5080, P1 CONN_01X02, P2 CONN_01X02, P3 CONN_01X02, U1 NCP1092, U2 LTM8050

Commit message: replace RJ45 output component and change some footprints association
Parts:
- removed J2: RJHSE-5080, symbol RJ45
- added J2: RJHSE-5080, symbol RJ45-8
Connections:
- no-connect marks 7 -> 6
Changed lines of the file:
@@
-EESchema Schematic File Version 2  date Tue 10 Feb 2015 03:19:18 PM EST
+EESchema Schematic File Version 2  date Wed 11 Feb 2015 09:15:43 AM EST
 LIBS:power
 LIBS:device
@@
 LIBS:valves
 LIBS:onsemi
+LIBS:ltm-ps-cache
 EELAYER 25  0
 EELAYER END
@@
 Sheet 1 1
 Title ""
-Date "4 feb 2015"
+Date "11 feb 2015"
 Rev ""
 Comp ""
@@
 Comment4 ""
 $EndDescr
-NoConn ~ 10800 6950
+$Comp
+L RJ45-8 J2
+U 1 1 54DB63BE
+P 10450 6400
+F 0 "J2" V 10000 6150 60  0000 C CNN
+F 1 "RJHSE-5080" V 10900 6500 60  0000 C CNN
+	1    10450 6400
+	0    1    1    0
+$EndComp
 Text Notes 10675 7000 2    60   ~ 0
 Farnell - 1860577
@@
 Text Label 9900 6050 2    60   ~ 0
 TRD1+
-$Comp
-L RJ45 J2
-U 1 1 54D1E09D
-P 10450 6400
-F 0 "J2" V 10000 6150 60  0000 C CNN
-F 1 "RJHSE-5080" V 10900 6400 60  0000 C CNN
-	1    10450 6400
-	0    1    1    0
-$EndComp
 Text Label 3450 5625 0    60   ~ 0
 TRD4-

Commit message: Delete old style PCB file. Create the initial PCB with new style and new KiCAD release
Parts:
- C1: footprint (none) -> Capacitors_SMD:C_2220
- C2: footprint (none) -> Capacitors_SMD:C_1210
- C3: footprint (none) -> Capacitors_SMD:C_0805
- D1: footprint (none) -> Diodes_SMD:Diode-SMC_Standard
- D2, D3: footprint (none) -> libcms:SDIP04
- D4: footprint (none) -> Diodes_SMD:Diode-SMA_Standard
- J1: footprint (none) -> connect:RJ45_GIGABIT-MAGJACK
- J2: footprint (none) -> connect:RJ45_8N
- JP1: footprint (none) -> Pin_Headers:Pin_Header_Straight_1x03
- P1, P2, P3: footprint (none) -> Pin_Headers:Pin_Header_Straight_1x02
- R1, R10, R11, R2, R3, R4, R5, R6, R7, R8, R9: footprint (none) -> Resistors_SMD:R_0805
- U1: footprint (none) -> SMD_Packages:SOIC-8-N
- U2: footprint (none) -> libcms:BGA70-linear_standard
Other:
- moved on the sheet: U2B

Commit message: review design: correct inverting RJ45 signals. Modify ltm feedback resistor from 89.4k to 90.9k. Add silkscreen text for jumper
Parts:
- R2: value 89.4k -> 90.9k
Other:
- note added: "R1 sets LTM8050 switching frequency to 400kHz\nR2 sets LTM8050 output voltage to 5.12V"
- note removed: "R1 sets LTM8050 switching frequency to 400kHz\nR2 sets LTM8050 output voltage to 5.2V"
Changed lines of the file:
@@
 Text Label 9150 6050 2    60   ~ 0
 TRD4+
+Text Label 9150 5850 2    60   ~ 0
+TRD3-
+Text Label 9150 5750 2    60   ~ 0
+TRD3+
 Text Label 9150 5950 2    60   ~ 0
-TRD3-
-Text Label 9150 5850 2    60   ~ 0
-TRD3+
-Text Label 9150 5750 2    60   ~ 0
 TRD2-
 Text Label 9150 5650 2    60   ~ 0
@@
 Auxiliary source input - 7.5V to 58V
 Text Notes 8300 4150 0    60   ~ 12
-R1 sets LTM8050 switching frequency to 400kHz\nR2 sets LTM8050 output voltage to 5.2V
+R1 sets LTM8050 switching frequency to 400kHz\nR2 sets LTM8050 output voltage to 5.12V
 Text Notes 7550 2800 0    60   ~ 12
 For the prototype version, this jumper allows to select\nwhich signal will enable the DC/DC converter.\n- NCP1092 PGOOD\n- VIN (VPORT_P/Auxiliary source)
@@
 P 8050 4100
 F 0 "R2" V 8130 4100 50  0000 C CNN
-F 1 "89.4k" V 8057 4101 50  0000 C CNN
+F 1 "90.9k" V 8057 4101 50  0000 C CNN
 F 2 "Resistors_SMD:R_0805" H 8050 4100 60  0001 C CNN
 F 3 "" H 8050 4100 60  0001 C CNN
